File: hil-boards/hil01/hil01.kicad_pcb (KiCad board)
At the start: 2 copper layers, 80 x 25 mm, 36 parts, among them J1 USB_C_Receptacle_USB2.0, J2 RJ25, J3 Conn_01x08_Male, J4 Conn_01x02_Male, J5 Conn_01x03_Male, U1 ADUM4160, U2 AMS1117-3.3, U3 CH340G, U4 MAX485E, Y1 Crystal

Commit message: updated rs485 footprint
Parts:
- removed J4: Conn_01x02_Male, Connector_PinHeader_2.54mm:PinHeader_1x02_P2.54mm_Vertical
- removed J5: Conn_01x03_Male, Connector_PinHeader_2.54mm:PinHeader_1x03_P2.54mm_Vertical
- removed RJ1, RJ2, RJ3: 0, Resistor_SMD:R_0805_2012Metric_Pad1.20x1.40mm_HandSolder
- removed U2: AMS1117-3.3, Package_TO_SOT_SMD:SOT-223-3_TabPin2
- added C9: 0.1uF, Capacitor_SMD:C_0805_2012Metric_Pad1.18x1.45mm_HandSolder, F.Cu at (150.0, 107.7)
- J3: value Conn_01x08_Male -> Conn_01x02_Female; footprint Connector_PinHeader_2.54mm:PinHeader_1x08_P2.54mm_Vertical -> Connector_Kefa:TerminalBlock_Kefa_1x02_P6.35mm_Horizontal
- U4: footprint Package_SO:SO-8_5.3x6.2mm_P1.27mm -> Package_SO:SO-8_3.9x4.9mm_P1.27mm
- moved J3 23.1 mm to (169.6, 126.1), turned to 90 degrees
- moved J2 4.98 mm to (168.6, 105.1)
- moved U4 1.22 mm to (150.8, 118.7)
Connections:
- C4 pad 1: Net-(C4-Pad1) -> VCC
- C5 pad 1: Net-(C5-Pad1) -> VCC
- J3 pad 1: GND2 -> unconnected-(J3-Pad1)
- J3 pad 2: /RX -> unconnected-(J3-Pad2)
- PS1 pad 5: Net-(C4-Pad1) -> VCC
- R7 pad 2: Net-(C4-Pad1) -> VCC
- U1 pad 16: Net-(C4-Pad1) -> VCC
- U3 pad 13: /DTR -> unconnected-(U3-Pad13)
- U3 pad 14: /RTS -> unconnected-(U3-Pad14)
- U3 pad 9: /CTS -> unconnected-(U3-Pad9)
- U4 pad 1: unconnected-(U4-Pad1) -> /RX
- U4 pad 2: unconnected-(U4-Pad2) -> VCC
- U4 pad 3: unconnected-(U4-Pad3) -> VCC
- U4 pad 4: unconnected-(U4-Pad4) -> /TX
Other:
- board text removed: "1"
- board text removed: "2"
- board text removed: "3"
- board text removed: "5 4 1"
- board text removed: "6"
- board text removed: "7"
- board text removed: "8"
