File: hil-boards/z_hil01/hil01.kicad_sch (KiCad schematic)
At the start: 34 parts, among them J1 USB_C_Receptacle_USB2.0, J2 Conn_01x03_Male, U1 ADUM4160, U2 MAX485E, U3 CH340G, Y1 Crystal

Commit message: all elements placed
Parts:
- removed J2: Conn_01x03_Male, TerminalBlock_4Ucon:TerminalBlock_4Ucon_1x03_P3.50mm_Horizontal, symbol Connector:Conn_01x03_Male
- removed JP1, JP2, JP3: Jumper_2_Open, Connector_PinHeader_2.54mm:PinHeader_1x02_P2.54mm_Vertical, symbol Jumper:Jumper_2_Open
- removed R10, R12: 560, Resistor_SMD:R_0805_2012Metric_Pad1.20x1.40mm_HandSolder, symbol Device:R
- removed R11: 120, Resistor_SMD:R_0805_2012Metric_Pad1.20x1.40mm_HandSolder, symbol Device:R
- removed U2: MAX485E, Package_SO:SOP-8_3.9x4.9mm_P1.27mm, symbol Interface_UART:MAX485E
- added J2: RJ25, Connector_RJ:RJ25_Wayconn_MJEA-660X1_Horizontal, symbol Connector:RJ25
- added J3: Conn_01x02_Female, Connector_Kefa:TerminalBlock_Kefa_1x02_P6.35mm_Horizontal, symbol Connector:Conn_01x02_Female
- added U4: MAX485E, Package_SO:SO-8_3.9x4.9mm_P1.27mm, symbol Interface_UART:MAX485E
- renumbered R9 to R11
Connections:
- net GND2: now also U4.5 (GND)
- net RX: now also U4.1 (RO)
- net TX: now also U4.4 (DI)
- net +5V renamed VCC
- net VCC: now also U4.2 (~{RE}), U4.3 (DE), U4.8 (VCC)
Other:
- title: HIL-01 ISOLATED USB TO RS485 -> HIL01 - ISOLATED USB TO RS485
- moved on the sheet: C5
