File: c-labelplates/c00_hillabelplate/c00_hillabelplate.kicad_pcb (KiCad board)
At the start: 2 copper layers, 43 x 8 mm, 4 parts

Commit message: fixed name number
Other:
- board text added: "C00_hillabelplate"
- board text removed: "A00_hillabelplate"
Changed lines of the file:
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@@
   (gr_line (start 100 108) (end 143 108) (layer "Edge.Cuts") (width 0.1))
   (gr_line (start 143 100) (end 143 108) (layer "Edge.Cuts") (width 0.1))
-  (gr_text "A00_hillabelplate" (at 133.477 106.807) (layer "B.SilkS")
+  (gr_text "C00_hillabelplate" (at 133.477 106.807) (layer "B.SilkS")
     (effects (font (size 1 1) (thickness 0.15)) (justify mirror))
   )
