File: b-hil-boards/b06_hil/b06.kicad_sch (KiCad schematic)
At the start: 15 parts, among them J1 Conn_01x08_Socket, J2 USB_C_Receptacle_PowerOnly_6P, J3 USB_C_Receptacle_PowerOnly_6P, SW1 SW_Push, U4 ESP32_C3_SuperMini, U5 OLED-128x64-I2C

Commit message: B06: finalize PCB routing and design data
Complete the routed layout in b06.kicad_pcb, align schematic and project
settings, refresh fp-info-cache and sym-lib-table, add FreeRouting exchange
files (b06.dsn, b06.rules, b06.ses), the INA219 datasheet asset, the
Connector_Improved library symbol, and KiCad automatic backup archives.
Parts:
- removed J1: Conn_01x08_Socket, TerminalBlock_DoubleLevel:TerminalBlock_DoubleLevel_2x04_P3.50mm_Horizontal, symbol Connector:Conn_01x08_Socket
- removed J2, J3: USB_C_Receptacle_PowerOnly_6P, Connector_USB:USB_C_Receptacle_HRO_TYPE-C-31-M-12, symbol Connector:USB_C_Receptacle_PowerOnly_6P
- added C1, C3, C5: C, Capacitor_SMD:CP_Elec_8x10.5, symbol Device:C
- added C2, C4, C6, C7, C8, C9: C, Capacitor_SMD:C_0805_2012Metric_Pad1.18x1.45mm_HandSolder, symbol Device:C
- added D1, D2, D4: LED, LED_SMD:LED_0805_2012Metric_Pad1.15x1.40mm_HandSolder, symbol Device:LED
- added F2, F3: Polyfuse, Fuse:Fuse_1206_3216Metric_Pad1.42x1.75mm_HandSolder, symbol Device:Polyfuse
- added J2, J3, J4, J5: USB_C_Receptacle_PowerOnly_6P_Improved, Connector_USB:USB_C_Receptacle_HRO_TYPE-C-31-M-12, symbol Connector_Improved:USB_C_Receptacle_PowerOnly_6P_Improved
- added J6: Conn_01x14_Socket, TerminalBlock_DoubleLevel:TerminalBlock_DoubleLevel_2x07_P3.50mm_Horizontal, symbol Connector:Conn_01x14_Socket
- added R11, R12, R13, R14, R4, R7: R, Resistor_SMD:R_0805_2012Metric_Pad1.20x1.40mm_HandSolder, symbol Device:R
- added R5, R6, R8: R, Resistor_SMD:R_2512_6332Metric_Pad1.40x3.35mm_HandSolder, symbol Device:R
- added U1, U2, U3: INA219AxD, Package_SO:SOIC-8_3.9x4.9mm_P1.27mm, symbol Sensor_Energy:INA219AxD
- F1: footprint (none) -> Fuse:Fuse_1206_3216Metric_Pad1.42x1.75mm_HandSolder
Connections:
- net +5V: now also F2.2, F3.2, J3.A4 (VBUS), J3.A9 (VBUS), J3.B4 (VBUS), J3.B9 (VBUS)
- net DEFAULTS: now also J6.6 (Pin_6)
- net DISP_SCL: now also J6.2 (Pin_2), U1.4 (SCL), U2.4 (SCL), U3.4 (SCL)
- net DISP_SDA: now also J6.4 (Pin_4), U1.3 (SDA), U2.3 (SDA), U3.2 (A0), U3.3 (SDA)
- net ERR_LED_EXT: now also J6.8 (Pin_8)
- net at F1.1: now also C1.1, C2.1, R12.1, R4.1, R6.2, U1.8 (IN+)
- net at R3.1: now also J3.A5 (CC1)
- net at R2.1: now also J3.B5 (CC2)
- net +3.3V: now reaches U4.14 (3V3)
- net +3.3V: now also C7.1, C8.1, C9.1, J6.1 (Pin_1), J6.7 (Pin_7), U1.5 (VS), U2.2 (A0), U2.5 (VS), U3.5 (VS)
- net GND1 renamed GND
- net GND: now also C1.2, C2.2, C3.2, C4.2, C5.2, C6.2, C7.2, C8.2, C9.2, D1.1 (K), D2.1 (K), D4.1 (K), J2.A1 (GND), J2.A12 (GND), J2.B1 (GND), J2.B12 (GND), J3.A1 (GND), J3.A12 (GND), J3.B1 (GND), J3.B12 (GND), J4.A1 (GND), J4.A12 (GND), J4.B1 (GND), J4.B12 (GND), J5.A1 (GND), J5.A12 (GND), J5.B1 (GND), J5.B12 (GND), J6.11 (Pin_11), J6.13 (Pin_13), J6.3 (Pin_3), J6.5 (Pin_5), J6.9 (Pin_9), U1.1 (A1), U1.2 (A0), U1.6 (GND), U2.1 (A1), U2.6 (GND), U3.1 (A1), U3.6 (GND)
- new net: J2.A4 (VBUS), J2.A9 (VBUS), J2.B4 (VBUS), J2.B9 (VBUS), R6.1, U1.7 (IN-)
- new net: C5.1, C6.1, F3.1, R11.1, R14.1, R8.2, U3.8 (IN+)
- new net: C3.1, C4.1, F2.1, R13.1, R5.2, R7.1, U2.8 (IN+)
- new net: J5.A4 (VBUS), J5.A9 (VBUS), J5.B4 (VBUS), J5.B9 (VBUS), R8.1, U3.7 (IN-)
- new net: D1.2 (A), R4.2
- new net: J4.A4 (VBUS), J4.A9 (VBUS), J4.B4 (VBUS), J4.B9 (VBUS), R5.1, U2.7 (IN-)
- new net: D4.2 (A), R11.2
- new net: D2.2 (A), R7.2
- new net OUT_PW_LED1: J6.10 (Pin_10), R12.2
- new net OUT_PW_LED2: J6.12 (Pin_12), R13.2
- new net OUT_PW_LED3: J6.14 (Pin_14), R14.2
- no-connect marks 10 -> 19
Other:
- note added: "0x40"
- note added: "0x41"
- note added: "0x42"
- moved on the sheet: F1, R2, R3, U4

Commit message: B06: add single-board Gerber outputs
Export gerber/single (copper, mask, paste, silkscreen, edge cuts, drills, and b06-single.zip) for one-up fabrication; refresh PCB, schematic, and project layout; rotate KiCad automatic backups.
Parts:
- renumbered J3 to J1, J5 to J2, J4 to J3, J2 to J4, J6 to J5
Changed lines of the file:
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@@
   (symbol (lib_id "Connector:Conn_01x14_Socket") (at 255.27 66.04 0) (mirror x) (unit 1)
     (in_bom yes) (on_board yes) (dnp no)
-    (property "Reference" "J6" (at 256.54 66.04 0)
+    (property "Reference" "J5" (at 256.54 66.04 0)
       (effects (font (size 1.27 1.27)) (justify left))
     )
@@
       (project "b06"
         (path "/f3c2aef5-4f0e-4b7a-b0f6-d797c84c763a"
-          (reference "J6") (unit 1)
+          (reference "J5") (unit 1)
         )
       )
@@
   (symbol (lib_name "USB_C_Receptacle_PowerOnly_6P_Improved_1") (lib_id "Connector_Improved:USB_C_Receptacle_PowerOnly_6P_Improved") (at 29.21 172.72 0) (unit 1)
     (in_bom yes) (on_board yes) (dnp no)
-    (property "Reference" "J3" (at 29.21 154.94 0)
+    (property "Reference" "J1" (at 29.21 154.94 0)
       (effects (font (size 1.27 1.27)))
     )
@@
       (project "b06"
         (path "/f3c2aef5-4f0e-4b7a-b0f6-d797c84c763a"
-          (reference "J3") (unit 1)
+          (reference "J1") (unit 1)
         )
       )
@@
   (symbol (lib_name "USB_C_Receptacle_PowerOnly_6P_Improved_1") (lib_id "Connector_Improved:USB_C_Receptacle_PowerOnly_6P_Improved") (at 30.48 31.75 0) (unit 1)
     (in_bom yes) (on_board yes) (dnp no)
-    (property "Reference" "J2" (at 30.48 13.97 0)
+    (property "Reference" "J4" (at 30.48 13.97 0)
       (effects (font (size 1.27 1.27)))
     )
@@
       (project "b06"
         (path "/f3c2aef5-4f0e-4b7a-b0f6-d797c84c763a"
-          (reference "J2") (unit 1)
+          (reference "J4") (unit 1)
         )
       )
@@
   (symbol (lib_name "USB_C_Receptacle_PowerOnly_6P_Improved_1") (lib_id "Connector_Improved:USB_C_Receptacle_PowerOnly_6P_Improved") (at 30.48 125.73 0) (unit 1)
     (in_bom yes) (on_board yes) (dnp no)
-    (property "Reference" "J5" (at 30.48 107.95 0)
+    (property "Reference" "J2" (at 30.48 107.95 0)
       (effects (font (size 1.27 1.27)))
     )
@@
       (project "b06"
         (path "/f3c2aef5-4f0e-4b7a-b0f6-d797c84c763a"
-          (reference "J5") (unit 1)
+          (reference "J2") (unit 1)
         )
       )
@@
   (symbol (lib_name "USB_C_Receptacle_PowerOnly_6P_Improved_1") (lib_id "Connector_Improved:USB_C_Receptacle_PowerOnly_6P_Improved") (at 30.48 78.74 0) (unit 1)
     (in_bom yes) (on_board yes) (dnp no)
-    (property "Reference" "J4" (at 30.48 60.96 0)
+    (property "Reference" "J3" (at 30.48 60.96 0)
       (effects (font (size 1.27 1.27)))
     )
@@
       (project "b06"
         (path "/f3c2aef5-4f0e-4b7a-b0f6-d797c84c763a"
-          (reference "J4") (unit 1)
-        )
-      )
+          (reference "J3") (unit 1)
+        )
+      )
