File: b-hil-boards/b06_hil/pcb/b06.kicad_pcb (KiCad board)
At the start: 2 copper layers, 100 x 50 mm, 52 parts, among them J1 USB_C_Receptacle_PowerOnly_6P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, J2 USB_C_Receptacle_PowerOnly_6P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, J3 USB_C_Receptacle_PowerOnly_6P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, J4 USB_C_Receptacle_PowerOnly_6P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, J5 Conn_01x14_Socket, SW1 SW_Push, U1 INA219AxD, U2 INA219AxD, U3 INA219AxD, U4 ESP32_C3_SuperMini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

Commit message: refactor(b06): move KiCad project into pcb/ subdirectory
Connections:
- D3 pad 2: +3V3 -> +3.3V
- R1 pad 1: +3V3 -> +3.3V
- U5 pad 2: +3V3 -> +3.3V
Routing:
- net +3.3V: track 150.4 -> 203.1 mm, vias 6 -> 8
- net +3V3: track 49.4 -> 0.00 mm, vias 2 -> 0
