File: b-hil-boards/b06_hil/pcb/b06.kicad_pcb (KiCad board)
At the start: 2 copper layers, 100 x 50 mm, 52 parts, among them J1 USB_C_Receptacle_PowerOnly_6P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, J2 USB_C_Receptacle_PowerOnly_6P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, J3 USB_C_Receptacle_PowerOnly_6P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, J4 USB_C_Receptacle_PowerOnly_6P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, J5 Conn_01x14_Socket, SW1 SW_Push, U1 INA219AxD, U2 INA219AxD, U3 INA219AxD, U4 ESP32_C3_SuperMini, U5 OLED-128x64-I2C

Commit message: feat(b06_hil): add external power-off switch and always-on solder jumper
Parts:
- added JP1: SolderJumper_2_Open, Jumper:SolderJumper-2_P1.3mm_Open_RoundedPad1.0x1.5mm, F.Cu at (160.4, 37.2)
- J5: value Conn_01x14_Socket -> Conn_01x16_Socket; footprint TerminalBlock_DoubleLevel:TerminalBlock_DoubleLevel_2x07_P3.50mm_Horizontal -> TerminalBlock_DoubleLevel:TerminalBlock_DoubleLevel_2x08_P3.50mm_Horizontal
- moved J5 3.50 mm to (175.6, 61.7)
Connections:
- J1 pad A4: +5V -> /PSWI
- J1 pad A9: +5V -> /PSWI
- J1 pad B4: +5V -> /PSWI
- J1 pad B9: +5V -> /PSWI
Routing:
- net /PSWI: track 0.00 -> 153.2 mm, vias 0 -> 2
- net +5V: track 97.0 -> 88.2 mm, vias 6 -> 5
- net +3.3V: track 203.1 -> 207.2 mm
- net /DEFAULTS: track 97.9 -> 102.0 mm
- net /ERR_LED_EXT: track 51.4 -> 47.7 mm
- net /DISP_SCL: track 118.8 -> 122.2 mm
- net /OUT_PW_LED2: track 88.2 -> 85.9 mm
- net /OUT_PW_LED3: track 110.1 -> 112.3 mm
- net /OUT_PW_LED1: track 76.7 -> 78.5 mm
Other:
- board text added: "PSWI"
- board text added: "PSWO"
- board text added: "PWR_SWI_IN"
- board text added: "PWR_SWI_OUT"
