File: b-hil-boards/b06_hil/pcb/b06.kicad_sch (KiCad schematic)
At the start: 43 parts, among them J1 USB_C_Receptacle_PowerOnly_6P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, J2 USB_C_Receptacle_PowerOnly_6P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, J3 USB_C_Receptacle_PowerOnly_6P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, J4 USB_C_Receptacle_PowerOnly_6P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, J5 Conn_01x14_Socket, SW1 SW_Push, U1 INA219AxD, U2 INA219AxD, U3 INA219AxD, U4 ESP32_C3_SuperMini, U5 OLED-128x64-I2C

Commit message: feat(b06_hil): add external power-off switch and always-on solder jumper
Parts:
- removed J5: Conn_01x14_Socket, TerminalBlock_DoubleLevel:TerminalBlock_DoubleLevel_2x07_P3.50mm_Horizontal, symbol Connector:Conn_01x14_Socket
- added J5: Conn_01x16_Socket, TerminalBlock_DoubleLevel:TerminalBlock_DoubleLevel_2x08_P3.50mm_Horizontal, symbol Connector:Conn_01x16_Socket
- added JP1: SolderJumper_2_Open, Jumper:SolderJumper-2_P1.3mm_Open_RoundedPad1.0x1.5mm, symbol Jumper:SolderJumper_2_Open
Connections:
- net +3.3V: now also J5.1 (Pin_1), J5.7 (Pin_7)
- net +5V: now also J5.16 (Pin_16), JP1.2 (B); no longer J1.A4 (VBUS), J1.A9 (VBUS), J1.B4 (VBUS), J1.B9 (VBUS)
- net DEFAULTS: now also J5.6 (Pin_6)
- net DISP_SCL: now also J5.2 (Pin_2)
- net DISP_SDA: now also J5.4 (Pin_4)
- net ERR_LED_EXT: now also J5.8 (Pin_8)
- net GND: now also J5.11 (Pin_11), J5.13 (Pin_13), J5.3 (Pin_3), J5.5 (Pin_5), J5.9 (Pin_9)
- net OUT_PW_LED1: now also J5.10 (Pin_10)
- net OUT_PW_LED2: now also J5.12 (Pin_12)
- net OUT_PW_LED3: now also J5.14 (Pin_14)
- new net PSWI: J1.A4 (VBUS), J1.A9 (VBUS), J1.B4 (VBUS), J1.B9 (VBUS), J5.15 (Pin_15), JP1.1 (A)
