File: d-faceplates/d04_hil_faceplate/d04_hil_faceplate.kicad_pcb (KiCad board)
At the start: 2 copper layers, 62.9 x 64 mm, 16 parts

Commit message: d04_hil_faceplate: finalize components and complete PCB routing
Place the remaining faceplate components and finish the definitive routing
on the d04_hil_faceplate PCB. Remove the outdated single-board SVG/drill
exports generated from the early layout and rotate KiCad automatic backups.
Parts:
- removed H10, H9: MountingHole_Pad, MountingHoleSmall:MountingHole_1.15_M1_Pad_BottomOnly
- moved REF** 18.9 mm to (158.4, 132.8)
- moved REF** 4.00 mm to (131.5, 145.5)
- moved REF** 1.47 mm to (130.0, 118.0)
Routing:
- net GND: track 261.9 -> 268.2 mm
Changed lines of the file:
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@@
-  )
-  (footprint "MountingHoleSmall:MountingHole_1.15_M1_Pad_BottomOnly" (layer "F.Cu")
-    (at 159.2875 134.1)
-    (descr "Mounting Hole 1.15 M1 ")
-    (tags "Mounting Hole 1.15 M1 ")
-    (property "Sheetfile" "d03_hil_faceplate.kicad_sch")
-    (property "Sheetname" "")
-    (property "ki_description" "Mounting Hole with connection")
-    (property "ki_keywords" "mounting hole")
-    (attr exclude_from_pos_files)
-    (fp_text reference "H10" (at 0 -2.75) (layer "F.SilkS") hide
-        (effects (font (size 1 1) (thickness 0.15)))
-    )
-    (fp_text value "MountingHole_Pad" (at 0 2.75) (layer "F.Fab")
-        (effects (font (size 1 1) (thickness 0.15)))
-    )
-    (fp_text user "${REFERENCE}" (at 0 0) (layer "F.Fab")
-        (effects (font (size 1 1) (thickness 0.15)))
-    )
-    (fp_circle (center 0 0) (end 1.75 0)
-      (stroke (width 0.15) (type solid)) (fill none) (layer "Cmts.User"))
-    (fp_circle (center 0 0) (end 2 0)
-      (stroke (width 0.05) (type solid)) (fill none) (layer "F.CrtYd"))
-    (pad "1" thru_hole circle (at 0 0) (size 1.4 1.4) (drill 1.15) (layers "*.Cu" "*.Mask")
-      (net 1 "GND") (pinfunction "1") (pintype "input"))
-    (pad "1" connect circle (at 0 0) (size 3 3) (layers "B.Cu" "B.Mask")
-      (net 1 "GND") (pinfunction "1") (pintype "input"))
-  )
-  (footprint "MountingHoleSmall:MountingHole_1.15_M1_Pad_BottomOnly" (layer "F.Cu")
-    (at 160.7875 129.9)
-    (descr "Mounting Hole 1.15 M1 ")
-    (tags "Mounting Hole 1.15 M1 ")
-    (property "Sheetfile" "d03_hil_faceplate.kicad_sch")
-    (property "Sheetname" "")
-    (property "ki_description" "Mounting Hole with connection")
-    (property "ki_keywords" "mounting hole")
-    (attr exclude_from_pos_files)
-    (fp_text reference "H9" (at 0 -2.75) (layer "F.SilkS") hide
-        (effects (font (size 1 1) (thickness 0.15)))
-    )
-    (fp_text value "MountingHole_Pad" (at 0 2.75) (layer "F.Fab")
-        (effects (font (size 1 1) (thickness 0.15)))
-    )
-    (fp_text user "${REFERENCE}" (at 0 0) (layer "F.Fab")
-        (effects (font (size 1 1) (thickness 0.15)))
-    )
-    (fp_circle (center 0 0) (end 1.75 0)
-      (stroke (width 0.15) (type solid)) (fill none) (layer "Cmts.User"))
-    (fp_circle (center 0 0) (end 2 0)
-      (stroke (width 0.05) (type solid)) (fill none) (layer "F.CrtYd"))
-    (pad "1" thru_hole circle (at 0 0) (size 1.4 1.4) (drill 1.15) (layers "*.Cu" "*.Mask")
-      (net 1 "GND") (pinfunction "1") (pintype "input"))
-    (pad "1" connect circle (at 0 0) (size 3 3) (layers "B.Cu" "B.Mask")
-      (net 1 "GND") (pinfunction "1") (pintype "input"))
   )
   (footprint "MountingHoleSmall:MountingHole_1.15_M1_Pad_BottomOnly" (layer "F.Cu")
@@
   )
   (footprint "MountingHoleDisplay:48×29 panel display" (layer "F.Cu")
-    (at 131.46875 118)
+    (at 130 118)
     (attr through_hole)
     (fp_text reference "REF**" (at -7.62 12.7 unlocked) (layer "F.SilkS") hide
@@
   )
   (footprint "MountingHoleConnector:15EDGWC-3mm81-Pluggable-Terminal-Block-Connector-5P" (layer "F.Cu")
-    (at 131.46875 141.5)
+    (at 131.46875 145.5)
     (attr through_hole)
     (fp_text reference "REF**" (at -7.62 12.7 unlocked) (layer "F.SilkS") hide
@@
   )
   (footprint "MountingHoleSwitch:DS-402_7mm_push_switch" (layer "F.Cu")
-    (at 172.75 120.5)
+    (at 158.4 132.75)
     (descr "Mounting Hole 5mm, no annular")
     (tags "mounting hole 5mm no annular")
     (attr exclude_from_pos_files exclude_from_bom)
-    (fp_text reference "REF**" (at 0 -6) (layer "F.SilkS")
+    (fp_text reference "REF**" (at 0 -6) (layer "F.SilkS") hide
         (effects (font (size 1 1) (thickness 0.15)))
     )
@@
   (gr_line (start 128.96875 132) (end 133.96875 132)
     (stroke (width 0.1) (type default)) (layer "Cmts.User"))
+  (gr_line (start 90 154) (end 172.9375 154)
+    (stroke (width 0.1) (type dot)) (layer "Cmts.User"))
   (gr_line (start 168.7375 127.8) (end 168.7375 136.2)
     (stroke (width 0.1) (type default)) (layer "Cmts.User"))
@@
   (segment (start 102.15 131.4) (end 103.65 129.9) (width 0.2) (layer "F.Cu") (net 1))
   (segment (start 161 154.5) (end 160.5 155) (width 0.2) (layer "F.Cu") (net 1))
+  (segment (start 156 138.75) (end 154.25 137) (width 0.2) (layer "F.Cu") (net 1))
   (segment (start 103.65 129.9) (end 103.65 110.5) (width 0.2) (layer "F.Cu") (net 1))
   (segment (start 160.45 104.8) (end 161 105.35) (width 0.2) (layer "F.Cu") (net 1))
   (segment (start 159.2875 153.5) (end 160.7875 155) (width 0.2) (layer "F.Cu") (net 1))
   (segment (start 160.7875 104.8) (end 160.7875 107.5) (width 0.2) (layer "F.Cu") (net 1))
+  (segment (start 159.2875 138.75) (end 156 138.75) (width 0.2) (layer "F.Cu") (net 1))
+  (segment (start 154.25 137) (end 154.25 129.25) (width 0.2) (layer "F.Cu") (net 1))
   (segment (start 103.65 107.5) (end 103.65 104.8) (width 0.2) (layer "F.Cu") (net 1))
   (segment (start 102.15 134.1) (end 130.9 134.1) (width 0.2) (layer "F.Cu") (net 1))
@@
   (segment (start 102.15 134.1) (end 102.15 131.4) (width 0.2) (layer "F.Cu") (net 1))
   (segment (start 159.2875 159.2) (end 102.15 159.2) (width 0.2) (layer "F.Cu") (net 1))
-  (segment (start 160.7875 132.6) (end 159.2875 134.1) (width 0.2) (layer "F.Cu") (net 1))
+  (segment (start 159.2875 138.75) (end 159.2875 153.5) (width 0.2) (layer "F.Cu") (net 1))
   (segment (start 160.7875 155) (end 160.7875 157.7) (width 0.2) (layer "F.Cu") (net 1))
-  (segment (start 159.2875 128.4) (end 160.7875 129.9) (width 0.2) (layer "F.Cu") (net 1))
   (segment (start 160.7875 157.7) (end 159.2875 159.2) (width 0.2) (layer "F.Cu") (net 1))
-  (segment (start 160.7875 129.9) (end 160.7875 132.6) (width 0.2) (layer "F.Cu") (net 1))
-  (segment (start 159.2875 134.1) (end 159.2875 153.5) (width 0.2) (layer "F.Cu") (net 1))
+  (segment (start 156.75 126.75) (end 159.2875 126.75) (width 0.2) (layer "F.Cu") (net 1))
+  (segment (start 154.25 129.25) (end 156.75 126.75) (width 0.2) (layer "F.Cu") (net 1))
   (segment (start 102.15 159.2) (end 102.15 156.5) (width 0.2) (layer "F.Cu") (net 1))
+  (segment (start 159.2875 126.75) (end 159.2875 109) (width 0.2) (layer "F.Cu") (net 1))
   (segment (start 103.65 110.5) (end 102.15 109) (width 0.2) (layer "F.Cu") (net 1))
-  (segment (start 159.2875 109) (end 159.2875 128.4) (width 0.2) (layer "F.Cu") (net 1))
   (segment (start 103.65 155) (end 103.65 135.6) (width 0.2) (layer "F.Cu") (net 1))
   (via (at 160.75 119.5) (size 0.6) (drill 0.3) (layers "F.Cu" "B.Cu") (free) (net 1))
